File: PCB's/In_out V2/IO.kicad_pcb (KiCad board)
At the start: 2 copper layers, 51.7 x 42.3 mm, 18 parts, among them J1 Conn_01x01_Pin, J2 Conn_01x02_Pin, J3 Conn_01x02_Pin, U1 L7805

Commit message: new pcbs
Connections:
- B1 pad T: Net-(Out3-Pin_2) -> /B
- Out3 pad 2: Net-(Out3-Pin_2) -> /B
Routing:
- net /B: track 0.00 -> 21.8 mm
- net Net-(Out3-Pin_2): track 10.4 -> 0.00 mm
Changed lines of the file:
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@@
   (net 15 "Net-(QL1-G)")
   (net 16 "Net-(B1-PadRN)")
-  (net 17 "Net-(Out3-Pin_2)")
-  (net 18 "Net-(Out2-Pin_3)")
-  (net 19 "Net-(Out3-Pin_3)")
+  (net 17 "Net-(Out2-Pin_3)")
+  (net 18 "Net-(Out3-Pin_3)")
   (footprint "Connector_Audio:Jack_6.35mm_Neutrik_NMJ6HFD3_Horizontal" (layer "F.Cu")
     (at 169.475 80.385)
@@
       (stroke (width 0.1) (type solid)) (layer "F.Fab"))
     (pad "R" thru_hole circle (at 6.35 0) (size 3 3) (drill 1.4) (layers "*.Cu" "*.Mask")
-      (net 19 "Net-(Out3-Pin_3)") (pintype "passive"))
+      (net 18 "Net-(Out3-Pin_3)") (pintype "passive"))
     (pad "RN" thru_hole circle (at 6.35 16.23) (size 3 3) (drill 1.4) (layers "*.Cu" "*.Mask")
       (net 16 "Net-(B1-PadRN)") (pintype "passive"))
@@
       (net 16 "Net-(B1-PadRN)") (pintype "passive"))
     (pad "T" thru_hole circle (at 0 0) (size 3 3) (drill 1.4) (layers "*.Cu" "*.Mask")
-      (net 17 "Net-(Out3-Pin_2)") (pintype "passive"))
+      (net 7 "/B") (pintype "passive"))
     (pad "TN" thru_hole circle (at 0 16.23) (size 3 3) (drill 1.4) (layers "*.Cu" "*.Mask")
       (net 16 "Net-(B1-PadRN)") (pintype "passive"))
@@
     (property "ki_keywords" "R res resistor")
     (attr through_hole)
-    (fp_text reference "RPD1" (at 3.81 -3.6) (layer "F.SilkS")
+    (fp_text reference "RPD1" (at 3.81 0) (layer "F.SilkS")
         (effects (font (size 1 1) (thickness 0.15)))
     )
@@
       (stroke (width 0.1) (type solid)) (layer "F.Fab"))
     (pad "R" thru_hole circle (at 6.35 0) (size 3 3) (drill 1.4) (layers "*.Cu" "*.Mask")
-      (net 18 "Net-(Out2-Pin_3)") (pintype "passive"))
+      (net 17 "Net-(Out2-Pin_3)") (pintype "passive"))
     (pad "RN" thru_hole circle (at 6.35 16.23) (size 3 3) (drill 1.4) (layers "*.Cu" "*.Mask")
       (net 6 "Net-(A1-PadRN)") (pintype "passive"))
@@
     (property "ki_keywords" "R res resistor")
     (attr through_hole)
-    (fp_text reference "RGate1" (at 3.81 -3.6) (layer "F.SilkS")
+    (fp_text reference "RGate1" (at 3.81 0) (layer "F.SilkS")
         (effects (font (size 1 1) (thickness 0.15)))
     )
@@
       (net 5 "/Signal_Gnd") (pinfunction "Pin_1") (pintype "passive"))
     (pad "2" thru_hole oval (at 0 -2.54 270) (size 1.7 1.7) (drill 1) (layers "*.Cu" "*.Mask")
-      (net 17 "Net-(Out3-Pin_2)") (pinfunction "Pin_2") (pintype "passive"))
+      (net 7 "/B") (pinfunction "Pin_2") (pintype "passive"))
     (pad "3" thru_hole oval (at 0 -5.08 270) (size 1.7 1.7) (drill 1) (layers "*.Cu" "*.Mask")
-      (net 19 "Net-(Out3-Pin_3)") (pinfunction "Pin_3") (pintype "passive"))
+      (net 18 "Net-(Out3-Pin_3)") (pinfunction "Pin_3") (pintype "passive"))
     (model "${KICAD6_3DMODEL_DIR}/Connector_PinHeader_2.54mm.3dshapes/PinHeader_1x03_P2.54mm_Vertical.wrl"
       (offset (xyz 0 0 0))
@@
       (net 4 "/A") (pinfunction "Pin_2") (pintype "passive"))
     (pad "3" thru_hole oval (at 0 -5.08 270) (size 1.7 1.7) (drill 1) (layers "*.Cu" "*.Mask")
-      (net 18 "Net-(Out2-Pin_3)") (pinfunction "Pin_3") (pintype "passive"))
+      (net 17 "Net-(Out2-Pin_3)") (pinfunction "Pin_3") (pintype "passive"))
     (model "${KICAD6_3DMODEL_DIR}/Connector_PinHeader_2.54mm.3dshapes/PinHeader_1x03_P2.54mm_Vertical.wrl"
       (offset (xyz 0 0 0))
@@
   (segment (start 175.825 117.365) (end 182.175 117.365) (width 0.25) (layer "F.Cu") (net 6))
   (segment (start 169.475 117.365) (end 175.825 117.365) (width 0.25) (layer "F.Cu") (net 6))
+  (segment (start 168.9175 79.8275) (end 169.475 80.385) (width 0.25) (layer "F.Cu") (net 7))
+  (segment (start 158.3625 79.8275) (end 168.9175 79.8275) (width 0.25) (layer "F.Cu") (net 7))
+  (segment (start 175.8 86.71) (end 175.8 88.2) (width 0.25) (layer "B.Cu") (net 7))
+  (segment (start 169.475 80.385) (end 175.8 86.71) (width 0.25) (layer "B.Cu") (net 7))
   (segment (start 136.79 89.4) (end 144.335 81.855) (width 0.25) (layer "B.Cu") (net 8))
   (segment (start 144.335 81.855) (end 144.335 81.2) (width 0.25) (layer "B.Cu") (net 8))
@@
   (segment (start 182.175 96.615) (end 175.825 96.615) (width 0.25) (layer "F.Cu") (net 16))
   (segment (start 169.475 96.615) (end 175.825 96.615) (width 0.25) (layer "F.Cu") (net 16))
-  (segment (start 175.8 86.71) (end 175.8 88.2) (width 0.25) (layer "B.Cu") (net 17))
-  (segment (start 169.475 80.385) (end 175.8 86.71) (width 0.25) (layer "B.Cu") (net 17))
-  (segment (start 178.125 103.435) (end 178.125 109) (width 0.25) (layer "B.Cu") (net 18))
-  (segment (start 175.825 101.135) (end 178.125 103.435) (width 0.25) (layer "B.Cu") (net 18))
-  (segment (start 175.825 80.385) (end 178.34 82.9) (width 0.25) (layer "B.Cu") (net 19))
-  (segment (start 178.34 82.9) (end 178.34 88.2) (width 0.25) (layer "B.Cu") (net 19))
+  (segment (start 178.125 103.435) (end 178.125 109) (width 0.25) (layer "B.Cu") (net 17))
+  (segment (start 175.825 101.135) (end 178.125 103.435) (width 0.25) (layer "B.Cu") (net 17))
+  (segment (start 175.825 80.385) (end 178.34 82.9) (width 0.25) (layer "B.Cu") (net 18))
+  (segment (start 178.34 82.9) (end 178.34 88.2) (width 0.25) (layer "B.Cu") (net 18))
 )
