File: PCB's/In_out V2/IO.kicad_sch (KiCad schematic)
At the start: 18 parts, among them J1 Conn_01x01_Pin, J2 Conn_01x02_Pin, J3 Conn_01x02_Pin, U1 L7805

Commit message: new pcbs
Connections:
- net B: now also B1.T, Out3.2 (Pin_2)
Changed lines of the file:
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@@
   (junction (at 62.23 123.19) (diameter 0) (color 0 0 0 0)
   )
+  (junction (at 153.67 66.04) (diameter 0) (color 0 0 0 0)
+  )
   (junction (at 137.16 127) (diameter 0) (color 0 0 0 0)
   )
@@
     (stroke (width 0) (type default))
   )
+  (wire (pts (xy 153.67 66.04) (xy 154.94 66.04))
+    (stroke (width 0) (type default))
+  )
