File: PCB's/Loop Board V3 Jackless/Loop Board 3 Jackless Input/Loop Board 3 Jackless Input.kicad_pcb (KiCad board)
At the start: 2 copper layers, 120.5 x 60 mm, 38 parts, among them J1 8P8C, J2 Conn_01x08_Pin, U1 L7805

Commit message: latest Version PCBs
Parts:
- J1: footprint Connector_RJ:RJ45_Amphenol_54602-x08_Horizontal -> Relay_parts:RJ456
- L/Mono1, R1: footprint Connector_Audio:Jack_6.35mm_Neutrik_NMJ6HCD2_Horizontal -> Relay_parts:0.25 Audio JAck
