File: PCB's/Loop Board V3 Jackless/Loop Board 3 Jackless Output/Loop Board 3 Jackless Output.kicad_pcb (KiCad board)
At the start: 2 copper layers, 120.5 x 60 mm, 33 parts, among them J2 Conn_01x08_Pin, U1 L7805

Commit message: latest Version PCBs
Parts:
- L/Mono1, R1: footprint Connector_Audio:Jack_6.35mm_Neutrik_NMJ6HCD2_Horizontal -> Relay_parts:0.25 Audio JAck
