File: PCB's/Control Board v2/Control Board v2.kicad_sch (KiCad schematic)
At the start: 13 parts, among them J1 Power In, J2 LED Strip Conn, J3 Expansion, J4 Expansion, U1 ESP32-DEVKITC-32E, U2 L7805

Commit message: updates
Connections:
- net GND: now also U1.J2_14 (GND_J2_14), U1.J3_1 (GND_J3_1)
- net LED_1_Data: no longer U1.J3_16 (IO15)
- net LED_2_Data: no longer U1.J2_15 (IO13)
- net LED_3_Data: no longer U1.J2_13 (IO12)
- new net LED_1_sig: U1.J3_16 (IO15)
- new net LED_2_sig: U1.J2_15 (IO13)
- new net LED_3_sig: U1.J2_13 (IO12)
Changed lines of the file:
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@@
   (junction (at 46.99 128.27) (diameter 0) (color 0 0 0 0)
   )
+  (wire (pts (xy 106.68 132.08) (xy 111.76 132.08))
+    (stroke (width 0) (type default))
+  )
   (wire (pts (xy 227.33 53.34) (xy 247.65 53.34))
     (stroke (width 0) (type default))
@@
     (stroke (width 0) (type default))
   )
+  (wire (pts (xy 106.68 143.51) (xy 106.68 132.08))
+    (stroke (width 0) (type default))
+  )
   (wire (pts (xy 41.91 87.63) (xy 41.91 88.9))
     (stroke (width 0) (type default))
@@
     (stroke (width 0) (type default))
   )
+  (wire (pts (xy 59.69 176.53) (xy 66.04 176.53))
+    (stroke (width 0) (type default))
+  )
   (wire (pts (xy 121.92 163.83) (xy 121.92 162.56))
     (stroke (width 0) (type default))
@@
     )
   )
-  (global_label "LED_1_Data" (shape input) (at 118.11 181.61 0) (fields_autoplaced)
+  (global_label "LED_1_sig" (shape input) (at 118.11 181.61 0) (fields_autoplaced)
     (effects (font (size 1.27 1.27)) (justify left))
-    (property "Intersheetrefs" "${INTERSHEET_REFS}" (at 131.9807 181.61 0)
+    (property "Intersheetrefs" "${INTERSHEET_REFS}" (at 130.4689 181.61 0)
       (effects (font (size 1.27 1.27)) (justify left) hide)
     )
   )
-  (global_label "LED_2_Data" (shape input) (at 49.53 179.07 180) (fields_autoplaced)
+  (global_label "LED_2_sig" (shape input) (at 49.53 179.07 180) (fields_autoplaced)
     (effects (font (size 1.27 1.27)) (justify right))
-    (property "Intersheetrefs" "${INTERSHEET_REFS}" (at 35.6593 179.07 0)
+    (property "Intersheetrefs" "${INTERSHEET_REFS}" (at 37.1711 179.07 0)
       (effects (font (size 1.27 1.27)) (justify right) hide)
     )
@@
     )
   )
-  (global_label "LED_3_Data" (shape input) (at 49.53 173.99 180) (fields_autoplaced)
+  (global_label "LED_3_sig" (shape input) (at 49.53 173.99 180) (fields_autoplaced)
     (effects (font (size 1.27 1.27)) (justify right))
-    (property "Intersheetrefs" "${INTERSHEET_REFS}" (at 35.6593 173.99 0)
+    (property "Intersheetrefs" "${INTERSHEET_REFS}" (at 37.1711 173.99 0)
       (effects (font (size 1.27 1.27)) (justify right) hide)
     )
@@
     )
   )
+  (symbol (lib_id "power:GND") (at 59.69 176.53 0) (unit 1)
+    (in_bom yes) (on_board yes) (dnp no) (fields_autoplaced)
+    (property "Reference" "#PWR049" (at 59.69 182.88 0)
+      (effects (font (size 1.27 1.27)) hide)
+    )
+    (property "Value" "GND" (at 59.69 181.61 0)
+      (effects (font (size 1.27 1.27)))
+    )
+    (property "Footprint" "" (at 59.69 176.53 0)
+      (effects (font (size 1.27 1.27)) hide)
+    )
+    (property "Datasheet" "" (at 59.69 176.53 0)
+      (effects (font (size 1.27 1.27)) hide)
+    )
+    (pin "1")
+    (instances
+      (project "Control Board v2"
+        (path "/3fc3ce26-f513-474c-a2f4-dd3cfa56ee8d"
+          (reference "#PWR049") (unit 1)
+        )
+      )
+    )
+  )
   (symbol (lib_id "power:GND") (at 265.43 88.9 0) (unit 1)
     (in_bom yes) (on_board yes) (dnp no) (fields_autoplaced)
@@
         )
       )
+    )
+  )
+  (symbol (lib_id "power:GND") (at 111.76 132.08 0) (unit 1)
+    (in_bom yes) (on_board yes) (dnp no) (fields_autoplaced)
+    (property "Reference" "#PWR048" (at 111.76 138.43 0)
+      (effects (font (size 1.27 1.27)) hide)
+    )
+    (property "Value" "GND" (at 111.76 137.16 0)
+      (effects (font (size 1.27 1.27)))
+    )
+    (property "Footprint" "" (at 111.76 132.08 0)
+      (effects (font (size 1.27 1.27)) hide)
+    )
+    (property "Datasheet" "" (at 111.76 132.08 0)
+      (effects (font (size 1.27 1.27)) hide)
+    )
+    (pin "1")
+    (instances
+      (project "Control Board v2"
+        (path "/3fc3ce26-f513-474c-a2f4-dd3cfa56ee8d"
+          (reference "#PWR048") (unit 1)
+        )
+      )
