File: PCB's/Control Board v2/LED.kicad_sch (KiCad schematic)
At the start: 9 parts, among them U3 TXS0101DBV

Commit message: updates
Parts:
- added RPD1_1 (x3): ~, Resistor_SMD:R_0805_2012Metric_Pad1.20x1.40mm_HandSolder, symbol Device:R
Connections:
- net LED_1_sig: now also RPD1_1.1
- net LED_2_sig: now also RPD1_1.1
- net LED_3_sig: now also RPD1_1.1
- net at LED1.3 (DIN), U3.4 (B): now also RPD1_1.2 (x3)
Changed lines of the file:
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@@
 (kicad_sch (version 20230121) (generator eeschema)
   (paper "A4")
+  (junction (at 88.9 151.13) (diameter 0) (color 0 0 0 0)
+  )
+  (junction (at 99.06 39.37) (diameter 0) (color 0 0 0 0)
+  )
+  (junction (at 49.53 102.87) (diameter 0) (color 0 0 0 0)
+  )
+  (junction (at 95.25 93.98) (diameter 0) (color 0 0 0 0)
+  )
+  (junction (at 50.8 162.56) (diameter 0) (color 0 0 0 0)
+  )
+  (junction (at 48.26 52.07) (diameter 0) (color 0 0 0 0)
+  )
   (wire (pts (xy 81.28 134.62) (xy 81.28 151.13))
     (stroke (width 0) (type default))
   )
+  (wire (pts (xy 49.53 102.87) (xy 49.53 97.79))
+    (stroke (width 0) (type default))
+  )
   (wire (pts (xy 139.7 27.94) (xy 142.24 27.94))
     (stroke (width 0) (type default))
   )
-  (wire (pts (xy 81.28 151.13) (xy 101.6 151.13))
+  (wire (pts (xy 81.28 151.13) (xy 88.9 151.13))
     (stroke (width 0) (type default))
   )
@@
     (stroke (width 0) (type default))
   )
+  (wire (pts (xy 83.82 104.14) (xy 95.25 104.14))
+    (stroke (width 0) (type default))
+  )
   (wire (pts (xy 80.01 77.47) (xy 80.01 93.98))
     (stroke (width 0) (type default))
   )
-  (wire (pts (xy 80.01 93.98) (xy 100.33 93.98))
+  (wire (pts (xy 80.01 93.98) (xy 95.25 93.98))
     (stroke (width 0) (type default))
   )
@@
     (stroke (width 0) (type default))
   )
+  (wire (pts (xy 48.26 52.07) (xy 53.34 52.07))
+    (stroke (width 0) (type default))
+  )
   (wire (pts (xy 87.63 27.94) (xy 99.06 27.94))
     (stroke (width 0) (type default))
@@
     (stroke (width 0) (type default))
   )
-  (wire (pts (xy 50.8 165.1) (xy 50.8 154.94))
+  (wire (pts (xy 50.8 154.94) (xy 50.8 162.56))
     (stroke (width 0) (type default))
   )
@@
     (stroke (width 0) (type default))
   )
-  (wire (pts (xy 48.26 53.34) (xy 48.26 43.18))
+  (wire (pts (xy 48.26 53.34) (xy 48.26 52.07))
+    (stroke (width 0) (type default))
+  )
+  (wire (pts (xy 81.28 171.45) (xy 81.28 161.29))
+    (stroke (width 0) (type default))
+  )
+  (wire (pts (xy 99.06 58.42) (xy 99.06 39.37))
+    (stroke (width 0) (type default))
+  )
+  (wire (pts (xy 50.8 162.56) (xy 50.8 165.1))
+    (stroke (width 0) (type default))
+  )
+  (wire (pts (xy 88.9 161.29) (xy 88.9 151.13))
     (stroke (width 0) (type default))
   )
@@
     (stroke (width 0) (type default))
   )
-  (wire (pts (xy 49.53 107.95) (xy 49.53 97.79))
+  (wire (pts (xy 49.53 107.95) (xy 49.53 102.87))
+    (stroke (width 0) (type default))
+  )
+  (wire (pts (xy 53.34 52.07) (xy 53.34 58.42))
     (stroke (width 0) (type default))
   )
@@
     (stroke (width 0) (type default))
   )
+  (wire (pts (xy 53.34 58.42) (xy 69.85 58.42))
+    (stroke (width 0) (type default))
+  )
   (wire (pts (xy 87.63 29.21) (xy 87.63 27.94))
     (stroke (width 0) (type default))
@@
     (stroke (width 0) (type default))
   )
+  (wire (pts (xy 88.9 151.13) (xy 101.6 151.13))
+    (stroke (width 0) (type default))
+  )
   (wire (pts (xy 149.86 130.81) (xy 149.86 132.08))
     (stroke (width 0) (type default))
   )
+  (wire (pts (xy 48.26 52.07) (xy 48.26 43.18))
+    (stroke (width 0) (type default))
+  )
+  (wire (pts (xy 55.88 162.56) (xy 55.88 171.45))
+    (stroke (width 0) (type default))
+  )
   (wire (pts (xy 60.96 158.75) (xy 60.96 154.94))
     (stroke (width 0) (type default))
@@
     (stroke (width 0) (type default))
   )
+  (wire (pts (xy 54.61 111.76) (xy 76.2 111.76))
+    (stroke (width 0) (type default))
+  )
+  (wire (pts (xy 55.88 171.45) (xy 81.28 171.45))
+    (stroke (width 0) (type default))
+  )
   (wire (pts (xy 142.24 21.59) (xy 143.51 21.59))
     (stroke (width 0) (type default))
   )
+  (wire (pts (xy 49.53 102.87) (xy 54.61 102.87))
+    (stroke (width 0) (type default))
+  )
+  (wire (pts (xy 54.61 102.87) (xy 54.61 111.76))
+    (stroke (width 0) (type default))
+  )
   (wire (pts (xy 60.96 166.37) (xy 60.96 177.8))
     (stroke (width 0) (type default))
@@
     (stroke (width 0) (type default))
   )
+  (wire (pts (xy 50.8 162.56) (xy 55.88 162.56))
+    (stroke (width 0) (type default))
+  )
   (wire (pts (xy 139.7 35.56) (xy 149.86 35.56))
     (stroke (width 0) (type default))
@@
     (stroke (width 0) (type default))
   )
+  (wire (pts (xy 76.2 111.76) (xy 76.2 104.14))
+    (stroke (width 0) (type default))
+  )
   (wire (pts (xy 38.1 30.48) (xy 33.02 30.48))
     (stroke (width 0) (type default))
@@
     (stroke (width 0) (type default))
   )
+  (wire (pts (xy 95.25 93.98) (xy 100.33 93.98))
+    (stroke (width 0) (type default))
+  )
   (wire (pts (xy 40.64 142.24) (xy 35.56 142.24))
     (stroke (width 0) (type default))
@@
   )
   (wire (pts (xy 34.29 85.09) (xy 34.29 83.82))
+    (stroke (width 0) (type default))
+  )
+  (wire (pts (xy 77.47 58.42) (xy 99.06 58.42))
+    (stroke (width 0) (type default))
+  )
+  (wire (pts (xy 95.25 104.14) (xy 95.25 93.98))
     (stroke (width 0) (type default))
   )
@@
     )
   )
+  (symbol (lib_id "Device:R") (at 80.01 104.14 90) (unit 1)
+    (in_bom yes) (on_board yes) (dnp no) (fields_autoplaced)
+    (property "Reference" "RPD1_1" (at 80.01 100.33 90)
+      (effects (font (size 1.27 1.27)))
+    )
+    (property "Value" "~" (at 80.01 100.33 90)
+      (effects (font (size 1.27 1.27)))
+    )
+    (property "Footprint" "Resistor_SMD:R_0805_2012Metric_Pad1.20x1.40mm_HandSolder" (at 80.01 105.918 90)
+      (effects (font (size 1.27 1.27)) hide)
+    )
+    (property "Datasheet" "~" (at 80.01 104.14 0)
+      (effects (font (size 1.27 1.27)) hide)
+    )
+    (pin "2")
+    (pin "1")
+    (instances
+      (project "Control Board v2"
+        (path "/3fc3ce26-f513-474c-a2f4-dd3cfa56ee8d/e2c63c3a-df9c-4a27-a62d-e65b06a25869"
+          (reference "RPD1_1") (unit 1)
+        )
+        (path "/3fc3ce26-f513-474c-a2f4-dd3cfa56ee8d/35332545-ffcd-4e75-8fd0-57173c91adb0"
+          (reference "BYP2") (unit 1)
+        )
+      )
+    )
+  )
   (symbol (lib_id "Logic_LevelTranslator:TXS0101DBV") (at 53.34 144.78 90) (unit 1)
     (in_bom yes) (on_board yes) (dnp no) (fields_autoplaced)
@@
     )
   )
+  (symbol (lib_id "Device:R") (at 73.66 58.42 90) (unit 1)
+    (in_bom yes) (on_board yes) (dnp no) (fields_autoplaced)
+    (property "Reference" "RPD1_1" (at 73.66 54.61 90)
+      (effects (font (size 1.27 1.27)))
+    )
+    (property "Value" "~" (at 73.66 54.61 90)
+      (effects (font (size 1.27 1.27)))
+    )
+    (property "Footprint" "Resistor_SMD:R_0805_2012Metric_Pad1.20x1.40mm_HandSolder" (at 73.66 60.198 90)
+      (effects (font (size 1.27 1.27)) hide)
+    )
+    (property "Datasheet" "~" (at 73.66 58.42 0)
+      (effects (font (size 1.27 1.27)) hide)
+    )
+    (pin "2")
+    (pin "1")
+    (instances
+      (project "Control Board v2"
+        (path "/3fc3ce26-f513-474c-a2f4-dd3cfa56ee8d/e2c63c3a-df9c-4a27-a62d-e65b06a25869"
+          (reference "RPD1_1") (unit 1)
+        )
+        (path "/3fc3ce26-f513-474c-a2f4-dd3cfa56ee8d/35332545-ffcd-4e75-8fd0-57173c91adb0"
+          (reference "BYP1") (unit 1)
+        )
+      )
+    )
+  )
   (symbol (lib_id "power:+5V") (at 33.02 29.21 0) (unit 1)
     (in_bom yes) (on_board yes) (dnp no) (fields_autoplaced)
@@
         )
       )
+    )
+  )
+  (symbol (lib_id "Device:R") (at 85.09 161.29 90) (unit 1)
+    (in_bom yes) (on_board yes) (dnp no) (fields_autoplaced)
+    (property "Reference" "RPD1_1" (at 85.09 157.48 90)
+      (effects (font (size 1.27 1.27)))
+    )
+    (property "Value" "~" (at 85.09 157.48 90)
+      (effects (font (size 1.27 1.27)))
+    )
+    (property "Footprint" "Resistor_SMD:R_0805_2012Metric_Pad1.20x1.40mm_HandSolder" (at 85.09 163.068 90)
+      (effects (font (size 1.27 1.27)) hide)
+    )
+    (property "Datasheet" "~" (at 85.09 161.29 0)
+      (effects (font (size 1.27 1.27)) hide)
+    )
+    (pin "2")
+    (pin "1")
+    (instances
+      (project "Control Board v2"
+        (path "/3fc3ce26-f513-474c-a2f4-dd3cfa56ee8d/e2c63c3a-df9c-4a27-a62d-e65b06a25869"
+          (reference "RPD1_1") (unit 1)
+        )
+        (path "/3fc3ce26-f513-474c-a2f4-dd3cfa56ee8d/35332545-ffcd-4e75-8fd0-57173c91adb0"
+          (reference "BYP3") (unit 1)
+        )
+      )
